File: plate/yamanami_keyboard_choc_top_plate.kicad_pcb (KiCad board)
At the start: 2 copper layers, 279.1 x 90 mm, 62 parts, among them SW2 KEY_SWITCH

Commit message: プレート修正
Parts:
- removed ? (x2): , Connector_PinSocket_1.00mm:PinSocket_1x02_P1.00mm_Vertical
- removed the Ref** at (375.7, 161.8)
- removed the Ref** at (180.4, 100.0)
- removed the Ref** at (298.6, 100.0)
- removed the Ref** at (103.4, 161.8)
- SW2: footprint kbd:SW_Hole_TH -> kbd:SW_Hole; moved to F.Cu
- SW2 (x47): footprint kbd:SW_Hole_TH -> kbd:SW_Hole
