File: cherry_mx/yamanami_keyboard.sch (KiCad schematic (older format))
At the start: 148 parts, among them J1 Breakaway_Tabs, J10 Conn_01x04, J11 Breakaway_Tabs, J12 Breakaway_Tabs, J13 Breakaway_Tabs, J14 Breakaway_Tabs, J2 Breakaway_Tabs, J3 Breakaway_Tabs, J4 Breakaway_Tabs, J5 Conn_02x03_Odd_Even, J6 USB_C_Receptacle_USB2.0, J7 Conn_01x04, J8 Conn_02x03_Odd_Even, J9 USB_C_Receptacle_USB2.0, SW1 SW_Push, U1 ATmega32U4-AU, U2 PRTR5V0U2X, U3 ATmega32U4-AU, U4 PRTR5V0U2X, Y1 16MHz, Y2 16MHz

Commit message: Cherry MX版のライブラリ整理
Parts:
- R1: symbol yamanami_keyboard-rescue:R-Device-yamanami_keyboard-rescue -> Device:R
- R4, R8: symbol yamanami_keyboard-rescue:R-Device-arch_keyboard-rescue -> Device:R
Changed lines of the file:
@@
 EESchema Schematic File Version 4
+LIBS:yamanami_keyboard-cache
 EELAYER 30 0
 EELAYER END
@@
 	995  1995 1075 1995
 $Comp
-L yamanami_keyboard-rescue:R-Device-yamanami_keyboard-rescue R1
+L Device:R R1
 U 1 1 5FA2159F
 P 4160 2360
@@
 $EndComp
 $Comp
-L yamanami_keyboard-rescue:+5V-power-yamanami_keyboard-rescue #PWR09
+L power:+5V #PWR09
 U 1 1 5FA4509E
 P 4160 2210
@@
 	4320 1560 4320 1695
 $Comp
-L yamanami_keyboard-rescue:+5V-power-yamanami_keyboard-rescue #PWR020
+L power:+5V #PWR020
 U 1 1 5FA71C9A
 P 3730 4870
@@
 	4080 3955 4300 3955
 $Comp
-L yamanami_keyboard-rescue:+5V-power-yamanami_keyboard-rescue #PWR014
+L power:+5V #PWR014
 U 1 1 5FAB4379
 P 4300 3925
@@
 $EndComp
 $Comp
-L Device:R R3
-U 1 1 5FBFC252
-P 5660 4890
-F 0 "R3" V 5570 4890 50  0000 C CNN
-F 1 "5.1k" V 5655 4890 50  0000 C CNN
-F 2 "Resistor_SMD:R_0603_1608Metric" V 5590 4890 50  0001 C CNN
-F 3 "~" H 5660 4890 50  0001 C CNN
-	1    5660 4890
-	0    -1   -1   0
-$EndComp
-$Comp
 L Device:R R6
 U 1 1 5FC6689D
@@
 $EndComp
 $Comp
-L yamanami_keyboard-rescue:R-Device-arch_keyboard-rescue R4
+L Device:R R4
 U 1 1 5FC9A64A
 P 2445 4295
@@
 	5510 2575 5510 2510
 Connection ~ 5510 2510
-$Comp
-L yamanami_keyboard-rescue:GND-power-arch_keyboard-rescue-yamanami_keyboard-rescue #PWR011
-U 1 1 5FBFE141
-P 5510 2890
-F 0 "#PWR011" H 5510 2640 50  0001 C CNN
-F 1 "GND" H 5515 2717 50  0000 C CNN
-F 2 "" H 5510 2890 50  0001 C CNN
-F 3 "" H 5510 2890 50  0001 C CNN
-	1    5510 2890
-	1    0    0    -1
-$EndComp
 Wire Wire Line
 	4915 2775 4915 2845
@@
 MOSI_R
 $Comp
-L yamanami_keyboard-rescue:+5VA-power-yamanami_keyboard-rescue #PWR044
+L power:+5VA #PWR044
 U 1 1 6009CA4A
 P 4255 9575
@@
 $EndComp
 $Comp
-L yamanami_keyboard-rescue:R-Device-arch_keyboard-rescue R8
+L Device:R R8
 U 1 1 6009CA98
 P 2800 9540
@@
 Connection ~ 5590 7950
 $Comp
-L yamanami_keyboard-rescue:GNDA-power-yamanami_keyboard-rescue #PWR038
+L power:GNDA #PWR038
 U 1 1 6009CB18
 P 5590 8330
@@
 	6190 8215 6190 8285
 $Comp
-L yamanami_keyboard-rescue:+5VA-power-yamanami_keyboard-rescue #PWR035
+L power:+5VA #PWR035
 U 1 1 6009CB45
 P 5590 7910
@@
 RESET_R
 $Comp
-L yamanami_keyboard-rescue:+5V-power-yamanami_keyboard-rescue #PWR08
+L power:+5V #PWR08
 U 1 1 5FBAA4E9
 P 5510 2450
@@
 	3730 4905 3730 4870
 $Comp
-L yamanami_keyboard-rescue:+5VA-power-yamanami_keyboard-rescue #PWR0101
+L power:+5VA #PWR0101
 U 1 1 5FF231DB
 P 3800 10405
@@
 $EndComp
 $Comp
-L yamanami_keyboard-rescue:VBUS-power-yamanami_keyboard-rescue #PWR046
+L power:VBUS #PWR046
 U 1 1 5FC65B7B
 P 6110 2510
@@
 	1    0    0    -1
 $EndComp
+$Comp
+L Device:R R3
+U 1 1 5FBFC252
+P 5660 4890
+F 0 "R3" V 5570 4890 50  0000 C CNN
+F 1 "5.1k" V 5655 4890 50  0000 C CNN
+F 2 "Resistor_SMD:R_0603_1608Metric" V 5590 4890 50  0001 C CNN
+F 3 "~" H 5660 4890 50  0001 C CNN
+	1    5660 4890
+	0    -1   -1   0
+$EndComp
+$Comp
+L power:GND #PWR011
+U 1 1 5FBFE141
+P 5510 2890
+F 0 "#PWR011" H 5510 2640 50  0001 C CNN
+F 1 "GND" H 5515 2717 50  0000 C CNN
+F 2 "" H 5510 2890 50  0001 C CNN
+F 3 "" H 5510 2890 50  0001 C CNN
+	1    5510 2890
+	1    0    0    -1
+$EndComp

Commit message: 回路図の変更完了（第一段）
Parts:
- removed C10, C9: 22pF, Capacitor_SMD:C_0603_1608Metric, symbol Device:C_Small
- removed C11, C12, C13: 0.1uF, Capacitor_SMD:C_0603_1608Metric, symbol Device:C_Small
- removed C15: 10uF, Capacitor_SMD:C_0603_1608Metric, symbol Device:C_Small
- removed C18: 1uF, Capacitor_SMD:C_0603_1608Metric, symbol Device:C_Small
- removed D50: D_Schottky_Small, Diode_SMD:D_SOD-123, symbol Device:D_Schottky_Small
- removed F2: 500mA, Fuse:Fuse_1206_3216Metric, symbol Device:Polyfuse
- removed J10, J7: Conn_01x04, random-keyboard-parts:PJ-3200B-4A-Assembly, symbol Connector_Generic:Conn_01x04
- removed J8: Conn_02x03_Odd_Even, Connector_PinHeader_2.54mm:PinHeader_2x03_P2.54mm_Vertical, symbol Connector_Generic:Conn_02x03_Odd_Even
- removed J9: USB_C_Receptacle_USB2.0, Type-C:HRO-TYPE-C-31-M-12-Assembly, symbol Type-C:HRO-TYPE-C-31-M-12
- removed R10, R11: 22, Resistor_SMD:R_0603_1608Metric, symbol Device:R
- removed R12, R9: 5.1k, Resistor_SMD:R_0603_1608Metric, symbol Device:R
- removed R7, R8: 10k, Resistor_SMD:R_0603_1608Metric, symbol Device:R
- removed RST2: RST_Jumper, Connector_PinSocket_2.54mm:PinSocket_1x02_P2.54mm_Vertical, symbol Device:Jumper
- removed U3: ATmega32U4-AU, Package_QFP:TQFP-44_10x10mm_P0.8mm, symbol MCU_Microchip_ATmega:ATmega32U4-AU
- removed U4: PRTR5V0U2X, random-keyboard-parts:SOT143B, symbol random-keyboard-parts:PRTR5V0U2X
- removed Y2: 16MHz, Crystal:Crystal_SMD_3225-4Pin_3.2x2.5mm, symbol Device:Crystal_GND24
- added J10, J11: USB_C_Receptacle, Connector_USB:USB_C_Receptacle_Amphenol_12401610E4-2A, symbol Connector:USB_C_Receptacle
- renumbered J6 to J01, J5 to J20, J1 to J90, J2 to J91, J3 to J92, J4 to J93, J11 to J94, J12 to J95, J13 to J96, J14 to J97
Connections:
- net MISO_R is gone; now on net row3: D43.1 (K), D44.1 (K), D45.1 (K), D46.1 (K), D47.1 (K), D48.1 (K)
- net SCK_R is gone; now on net col11: MX30.1 (COL), MX36.1 (COL), MX42.1 (COL), MX48.1 (COL)
- net col0_R is gone; now on net col6: MX25.1 (COL), MX31.1 (COL), MX37.1 (COL), MX43.1 (COL)
- net col1_R is gone; now on net col7: MX26.1 (COL), MX32.1 (COL), MX38.1 (COL), MX44.1 (COL)
- net col2_R is gone; now on net col8: MX27.1 (COL), MX33.1 (COL), MX39.1 (COL), MX45.1 (COL)
- net col3_R is gone; now on net col9: MX28.1 (COL), MX34.1 (COL), MX40.1 (COL), MX46.1 (COL)
- net col4_R is gone; now on net col10: MX29.1 (COL), MX35.1 (COL), MX41.1 (COL), MX47.1 (COL)
- net row0_R is gone; now on net row0: D25.1 (K), D26.1 (K), D27.1 (K), D28.1 (K), D29.1 (K), D30.1 (K)
- net row1_R is gone; now on net row1: D31.1 (K), D32.1 (K), D33.1 (K), D34.1 (K), D35.1 (K), D36.1 (K)
- net row2_R is gone; now on net row2: D37.1 (K), D38.1 (K), D39.1 (K), D40.1 (K), D41.1 (K), D42.1 (K)
- net row0: now also J10.A5 (CC1), J11.A5 (CC1)
- net row1: now also J10.B5 (CC2), J11.B5 (CC2)
- net row2: now also J10.A7 (D-), J10.B7 (D-), J11.A7 (D-), J11.B7 (D-)
- net row3: now also J10.A6 (D+), J10.B6 (D+), J11.A6 (D+), J11.B6 (D+)
- net col6: now reaches U1.26 (PD6)
- net col6: now also J10.B10 (RX1-), J10.B11 (RX1+), J11.B10 (RX1-), J11.B11 (RX1+)
- net col7: now reaches U1.27 (PD7)
- net col7: now also J10.A2 (TX1+), J10.A3 (TX1-), J11.A2 (TX1+), J11.A3 (TX1-)
- net col11: now reaches U1.38 (PF5)
- net col11: now also J10.B8 (SBU2), J11.B8 (SBU2)
- net col10: now reaches U1.39 (PF4)
- net col10: now also J10.A8 (SBU1), J11.A8 (SBU1)
- net col9: now reaches U1.40 (PF1)
- net col9: now also J10.B2 (TX2+), J10.B3 (TX2-), J11.B2 (TX2+), J11.B3 (TX2-)
- net col8: now reaches U1.41 (PF0)
- net col8: now also J10.A10 (RX2-), J10.A11 (RX2+), J11.A10 (RX2-), J11.A11 (RX2+)
- net DATA: no longer names the net of U1.20 (PD2)
- new net: J10.A1 (GND), J10.A12 (GND), J10.B1 (GND), J10.B12 (GND)
- new net: J10.A4 (VBUS), J10.A9 (VBUS), J10.B4 (VBUS), J10.B9 (VBUS)
- new net: J11.A1 (GND), J11.A12 (GND), J11.B1 (GND), J11.B12 (GND)
- new net: J11.A4 (VBUS), J11.A9 (VBUS), J11.B4 (VBUS), J11.B9 (VBUS)
- no-connect marks 40 -> 23
Other:
- note added: "ICSP"
- note added: "USB, ESD Protection, Polyfuse"
- note removed: "RIGHT HAND SCHEMATIC\n\nPower net changes:\nVCC -> VDD\nVBUS -> VDC\nGND -> GNDA\n+5V -> +5VA\nto prevent kicad from complaining about no connections between halves"
- note removed: "USB, ESD Protection,\nPolyfuse"
- moved on the sheet: C3, C4, C5, C7, D1, D10, D11, D12, D13, D14, D15, D16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
