File: cherry_mx/yamanami_keyboard.kicad_pcb (KiCad board)
At the start: 2 copper layers, 262.5 x 106.5 mm, 148 parts, among them J1 Breakaway_Tabs, J10 Conn_01x04, J11 Breakaway_Tabs, J12 Breakaway_Tabs, J13 Breakaway_Tabs, J14 Breakaway_Tabs, J2 Breakaway_Tabs, J3 Breakaway_Tabs, J4 Breakaway_Tabs, J5 Conn_02x03_Odd_Even, J6 USB_C_Receptacle_USB2.0, J7 Conn_01x04, J8 Conn_02x03_Odd_Even, J9 USB_C_Receptacle_USB2.0, SW1 SW_Push, U1 ATmega32U4-AU, U2 PRTR5V0U2X, U3 ATmega32U4-AU, U4 PRTR5V0U2X, Y1 16MHz, Y2 16MHz

Commit message: CherryMX版作成 ver.0.1
Parts:
- removed C1, C10, C2, C9: 22pF, Capacitor_SMD:C_0603_1608Metric
- removed C11, C12, C13, C3, C4, C5: 0.1uF, Capacitor_SMD:C_0603_1608Metric
- removed C15, C7: 10uF, Capacitor_SMD:C_0603_1608Metric
- removed C18, C8: 1uF, Capacitor_SMD:C_0603_1608Metric
- removed D49, D50: D_Schottky_Small, Diode_SMD:D_SOD-123
- removed F1, F2: 500mA, Fuse:Fuse_1206_3216Metric
- removed J1, J11, J12, J13, J14, J2, J3, J4: Breakaway_Tabs, random-keyboard-parts:breakaway-mousebites
- removed J10, J7: Conn_01x04, random-keyboard-parts:PJ-3200B-4A-Assembly
- removed J5, J8: Conn_02x03_Odd_Even, Connector_PinHeader_2.54mm:PinHeader_2x03_P2.54mm_Vertical
- removed J6, J9: USB_C_Receptacle_USB2.0, Type-C:HRO-TYPE-C-31-M-12-Assembly
- removed MX1, MX10, MX11, MX12, MX13, MX14, MX15, MX16, MX17, MX18, MX19, MX2, MX20, MX21, MX22, MX23, MX24, MX25, MX26, MX27, MX28, MX29, MX3, MX30, MX31, MX32, MX33, MX34, MX35, MX36, MX37, MX38, MX39, MX4, MX40, MX41, MX42, MX43, MX44, MX45, MX46, MX47, MX48, MX5, MX6, MX7, MX8, MX9: MX-noLED, MX_Only:MXOnly-1U-Hotswap
- removed R10, R11, R5, R6: 22, Resistor_SMD:R_0603_1608Metric
- removed R12, R3, R9: 5.1k, Resistor_SMD:R_0603_1608Metric
- removed R4, R7, R8: 10k, Resistor_SMD:R_0603_1608Metric
- removed RST2: RST_Jumper, Connector_PinSocket_2.54mm:PinSocket_1x02_P2.54mm_Vertical
- removed U3: ATmega32U4-AU, Package_QFP:TQFP-44_10x10mm_P0.8mm
- removed U4: PRTR5V0U2X, random-keyboard-parts:SOT143B
- removed Y1, Y2: 16MHz, Crystal:Crystal_SMD_3225-4Pin_3.2x2.5mm
- added G***: LOGO, 0-My_kbd_parts:icon, F.Cu at (68.9, 163.1)
- added G***: LOGO, 0-My_kbd_parts:icon_right_side, F.Cu at (295.1, 163.1)
- added G***: LOGO, 0-My_kbd_parts:icon, B.Cu at (68.9, 163.1)
- added G***: LOGO, 0-My_kbd_parts:icon_right_side, B.Cu at (295.1, 163.1)
- added H1: MountingHole, MountingHole:MountingHole_2.2mm_M2, F.Cu at (37.9, 83.9)
- added H10: MountingHole, MountingHole:MountingHole_2.2mm_M2, F.Cu at (152.9, 119.2)
- added H11: MountingHole, MountingHole:MountingHole_2.2mm_M2, F.Cu at (117.8, 159.3)
- added H12: MountingHole, MountingHole:MountingHole_2.2mm_M2, B.Cu at (117.8, 119.2)
- added H13: MountingHole, MountingHole:MountingHole_2.2mm_M2, F.Cu at (169.3, 141.1)
- added H14: MountingHole, MountingHole:MountingHole_2.2mm_M2, F.Cu at (76.3, 124.0)
- added H15: MountingHole, MountingHole:MountingHole_2.2mm_M2, F.Cu at (194.7, 141.1)
- added H16: MountingHole, MountingHole:MountingHole_2.2mm_M2, F.Cu at (246.1, 159.3)
- added H17: MountingHole, MountingHole:MountingHole_2.2mm_M2, F.Cu at (326.1, 83.9)
- added H18: MountingHole, MountingHole:MountingHole_2.2mm_M2, F.Cu at (326.1, 124.0)
- added H19: MountingHole, MountingHole:MountingHole_2.2mm_M2, F.Cu at (326.1, 164.1)
- added H2: MountingHole, MountingHole:MountingHole_2.2mm_M2, F.Cu at (37.9, 124.0)
- added H20: MountingHole, MountingHole:MountingHole_2.2mm_M2, F.Cu at (284.0, 164.1)
- added H21: MountingHole, MountingHole:MountingHole_2.2mm_M2, F.Cu at (245.9, 74.4)
- added H22: MountingHole, MountingHole:MountingHole_2.2mm_M2, F.Cu at (211.3, 79.1)
- added H23: MountingHole, MountingHole:MountingHole_2.2mm_M2, F.Cu at (76.0, 74.3)
- added H24: MountingHole, MountingHole:MountingHole_2.2mm_M2, F.Cu at (288.0, 124.0)
- added H25: MountingHole, MountingHole:MountingHole_2.2mm_M2, F.Cu at (246.1, 119.2)
- added H26: MountingHole, MountingHole:MountingHole_2.2mm_M2, F.Cu at (211.3, 119.2)
- added H3: MountingHole, MountingHole:MountingHole_2.2mm_M2, F.Cu at (37.9, 164.1)
- added H4: MountingHole, MountingHole:MountingHole_2.2mm_M2, F.Cu at (80.0, 164.1)
- added H5: MountingHole, MountingHole:MountingHole_2.2mm_M2, F.Cu at (165.3, 163.3)
- added H6: MountingHole, MountingHole:MountingHole_2.2mm_M2, F.Cu at (152.6, 79.1)
- added H7: MountingHole, MountingHole:MountingHole_2.2mm_M2, F.Cu at (118.1, 74.4)
- added H8: MountingHole, MountingHole:MountingHole_2.2mm_M2, F.Cu at (288.0, 74.4)
- added H9: MountingHole, MountingHole:MountingHole_2.2mm_M2, F.Cu at (198.6, 163.3)
- added OL1: OLED, 0-My_Parts:OLED_center_module_custom, F.Cu at (165.7, 97.6)
- added OL2: OLED, 0-My_Parts:OLED_center_module_custom, F.Cu at (198.3, 97.6)
- added REF**: , 0-My_Parts:mouse_bite, F.Cu at (271.6, 71.4)
- added REF**: , 0-My_Parts:mouse_bite, F.Cu at (92.3, 71.4)
- added REF**: , 0-My_Parts:mouse_bite, F.Cu at (306.6, 167.1)
- added REF**: , 0-My_Parts:mouse_bite, F.Cu at (57.4, 167.1)
- added SW10: SW_Push, 0-My_kbd_parts:CherryMX_Hotswap_via_1U_custom, F.Cu at (87.5, 104.9)
- added SW11: SW_Push, 0-My_kbd_parts:CherryMX_Hotswap_via_1U_custom, F.Cu at (87.5, 124.0)
- added SW12: SW_Push, 0-My_kbd_parts:CherryMX_Hotswap_via_1U_custom, F.Cu at (95.5, 149.6)
- added SW13: SW_Push, 0-My_kbd_parts:CherryMX_Hotswap_via_1U_custom, F.Cu at (106.6, 85.9)
- added SW14: SW_Push, 0-My_kbd_parts:CherryMX_Hotswap_via_1U_custom, F.Cu at (106.6, 104.9)
- added SW15: SW_Push, 0-My_kbd_parts:CherryMX_Hotswap_via_1U_custom, F.Cu at (106.6, 124.0)
- added SW16: SW_Push, 0-My_kbd_parts:CherryMX_Hotswap_via_1U_custom, F.Cu at (116.1, 147.8)
- added SW17: SW_Push, 0-My_kbd_parts:CherryMX_Hotswap_via_1U_custom, F.Cu at (125.6, 90.6)
- added SW18: SW_Push, 0-My_kbd_parts:CherryMX_Hotswap_via_1U_custom, F.Cu at (125.6, 109.7)
- added SW19: SW_Push, 0-My_kbd_parts:CherryMX_Hotswap_via_1U_custom, F.Cu at (125.6, 128.7)
- added SW2: SW_Push, 0-My_kbd_parts:CherryMX_Hotswap_via_1U_custom, F.Cu at (49.4, 114.5)
- added SW20: SW_Push, 0-My_kbd_parts:CherryMX_Hotswap_via_1U_custom, F.Cu at (135.2, 147.8)
- added SW21: SW_Push, 0-My_kbd_parts:CherryMX_Hotswap_via_1U_custom, F.Cu at (144.7, 90.6)
- added SW22: SW_Push, 0-My_kbd_parts:CherryMX_Hotswap_via_1U_custom, F.Cu at (144.7, 109.7)
- added SW23: SW_Push, 0-My_kbd_parts:CherryMX_Hotswap_via_1U_custom, F.Cu at (144.7, 128.7)
- added SW24: SW_Push, 0-My_kbd_parts:CherryMX_Hotswap_via_1U_custom, F.Cu at (155.7, 149.6)
- added SW25: SW_Push, 0-My_kbd_parts:CherryMX_Hotswap_via_1U_custom, F.Cu at (219.3, 90.6)
- added SW26: SW_Push, 0-My_kbd_parts:CherryMX_Hotswap_via_1U_custom, F.Cu at (219.3, 109.7)
- added SW27: SW_Push, 0-My_kbd_parts:CherryMX_Hotswap_via_1U_custom, F.Cu at (219.3, 128.7)
- added SW28: SW_Push, 0-My_kbd_parts:CherryMX_Hotswap_via_1U_custom, F.Cu at (208.2, 149.6)
- added SW29: SW_Push, 0-My_kbd_parts:CherryMX_Hotswap_via_1U_custom, F.Cu at (238.3, 90.6)
- added SW3: SW_Push, 0-My_kbd_parts:CherryMX_Hotswap_via_1U_custom, F.Cu at (49.4, 133.5)
- added SW30: SW_Push, 0-My_kbd_parts:CherryMX_Hotswap_via_1U_custom, F.Cu at (238.3, 109.7)
- added SW31: SW_Push, 0-My_kbd_parts:CherryMX_Hotswap_via_1U_custom, F.Cu at (238.3, 128.7)
- added SW32: SW_Push, 0-My_kbd_parts:CherryMX_Hotswap_via_1U_custom, F.Cu at (228.8, 147.8)
- added SW33: SW_Push, 0-My_kbd_parts:CherryMX_Hotswap_via_1U_custom, F.Cu at (257.4, 85.9)
- added SW34: SW_Push, 0-My_kbd_parts:CherryMX_Hotswap_via_1U_custom, F.Cu at (257.4, 104.9)
- added SW35: SW_Push, 0-My_kbd_parts:CherryMX_Hotswap_via_1U_custom, F.Cu at (257.4, 124.0)
- added SW36: SW_Push, 0-My_kbd_parts:CherryMX_Hotswap_via_1U_custom, F.Cu at (247.9, 147.8)
- added SW37: SW_Push, 0-My_kbd_parts:CherryMX_Hotswap_via_1U_custom, F.Cu at (276.4, 85.9)
- added SW38: SW_Push, 0-My_kbd_parts:CherryMX_Hotswap_via_1U_custom, F.Cu at (276.4, 104.9)
- added SW39: SW_Push, 0-My_kbd_parts:CherryMX_Hotswap_via_1U_custom, F.Cu at (276.4, 124.0)
- added SW4: SW_Push, 0-My_kbd_parts:CherryMX_Hotswap_via_1U_custom, F.Cu at (49.4, 152.6)
- added SW40: SW_Push, 0-My_kbd_parts:CherryMX_Hotswap_via_1U_custom, F.Cu at (268.4, 149.6)
- added SW41: SW_Push, 0-My_kbd_parts:CherryMX_Hotswap_via_1U_custom, F.Cu at (295.5, 95.4)
- added SW42: SW_Push, 0-My_kbd_parts:CherryMX_Hotswap_via_1U_custom, F.Cu at (295.5, 114.4)
- added SW43: SW_Push, 0-My_kbd_parts:CherryMX_Hotswap_via_1U_custom, F.Cu at (295.5, 133.5)
- added SW44: SW_Push, 0-My_kbd_parts:CherryMX_Hotswap_via_1U_custom, F.Cu at (295.5, 152.5)
- added SW45: SW_Push, 0-My_kbd_parts:CherryMX_Hotswap_via_1U_custom, F.Cu at (314.5, 95.4)
- added SW46: SW_Push, 0-My_kbd_parts:CherryMX_Hotswap_via_1U_custom, F.Cu at (314.5, 114.4)
- added SW47: SW_Push, 0-My_kbd_parts:CherryMX_Hotswap_via_1U_custom, F.Cu at (314.5, 133.5)
- added SW48: SW_Push, 0-My_kbd_parts:CherryMX_Hotswap_via_1U_custom, F.Cu at (314.5, 152.5)
- added SW49: SW_DIP_x04, 0-My_kbd_parts:DIP_SWITCH_EDS102SZ-4P, F.Cu at (165.7, 123.5)
- added SW5: SW_Push, 0-My_kbd_parts:CherryMX_Hotswap_via_1U_custom, F.Cu at (68.5, 95.4)
- added SW6: SW_Push, 0-My_kbd_parts:CherryMX_Hotswap_via_1U_custom, F.Cu at (68.5, 114.5)
- added SW7: SW_Push, 0-My_kbd_parts:CherryMX_Hotswap_via_1U_custom, F.Cu at (68.5, 133.5)
- added SW8: SW_Push, 0-My_kbd_parts:CherryMX_Hotswap_via_1U_custom, F.Cu at (68.5, 152.6)
- added SW9: SW_Push, 0-My_kbd_parts:CherryMX_Hotswap_via_1U_custom, F.Cu at (87.5, 85.9)
- added trrs1: TRRS, 0-My_kbd_parts:TRRS_PJ-320A, F.Cu at (170.6, 134.9)
- added trrs2: TRRS, 0-My_kbd_parts:TRRS_PJ-320A, F.Cu at (193.3, 134.9)
- D1, D10, D11, D12, D13, D14, D15, D16, D17, D18, D19, D2, D20, D21, D22, D23, D24, D25, D26, D27, D28, D29, D3, D30, D31, D32, D33, D34, D35, D36, D37, D38, D39, D4, D40, D41, D42, D43, D44, D45, D46, D47, D48, D5, D6, D7, D8, D9: footprint Diode_SMD:D_SOD-123 -> 0-My_Parts:D_SOD-123_custom
- R1: value 10k -> 4.7k
- R2: value 5.1k -> 4.7k
- SW1: footprint Connector_PinSocket_2.54mm:PinSocket_1x02_P2.54mm_Vertical -> 0-My_kbd_parts:CherryMX_Hotswap_via_1U_custom; moved to F.Cu
- U1: value ATmega32U4-AU -> RP2040-Zero; footprint Package_QFP:TQFP-44_10x10mm_P0.8mm -> 0-My_Parts:waveshare_rp2040-zero-Conthrough; moved to F.Cu
- U2: value PRTR5V0U2X -> RP2040-Zero; footprint random-keyboard-parts:SOT143B -> 0-My_Parts:waveshare_rp2040-zero-Conthrough; moved to F.Cu
- moved SW1 130.8 mm to (49.4, 95.4)
- moved D4 123.9 mm to (57.6, 154.8)
- moved D6 115.4 mm to (76.7, 116.6)
- moved D5 112.6 mm to (76.7, 97.6)
- moved D12 106.8 mm to (104.0, 150.6), turned to 100 degrees
- moved D3 98.9 mm to (57.6, 135.7)
- moved D36 98.2 mm to (256.0, 150.1)
- moved D28 95.6 mm to (217.1, 150.6), turned to 100 degrees
- moved D11 93.9 mm to (95.7, 126.1)
- moved D30 90.3 mm to (246.5, 111.9), turned to 90 degrees
- moved R2 88.5 mm to (197.1, 123.7), turned to 0 degrees
- moved U2 82.4 mm to (198.3, 89.2), turned to 0 degrees
- moved D21 77.6 mm to (152.9, 92.8)
- moved D45 77.5 mm to (322.7, 97.6), turned to 90 degrees
- moved D17 76.0 mm to (133.8, 92.8)
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Connections:
- D1 pad 2: Net-(D1-Pad2) -> Net-(D1-A)
- D11 pad 1: row1 -> row2
- D12 pad 1: row1 -> row3
- D13 pad 1: row2 -> row0
- D14 pad 1: row2 -> row1
- D16 pad 1: row2 -> row3
- D17 pad 1: row2 -> row0
- D18 pad 1: row2 -> row1
- D19 pad 1: row3 -> row2
- D2 pad 1: row0 -> row1
- D21 pad 1: row3 -> row0
- D22 pad 1: row3 -> row1
- D23 pad 1: row3 -> row2
- D25 pad 1: row0_R -> row0_r
- D26 pad 1: row0_R -> row1_r
- D27 pad 1: row0_R -> row2_r
- D28 pad 1: row0_R -> row3_r
- D29 pad 1: row0_R -> row0_r
- D3 pad 1: row0 -> row2
- D30 pad 1: row0_R -> row1_r
- D31 pad 1: row1_R -> row2_r
- D32 pad 1: row1_R -> row3_r
- D33 pad 1: row1_R -> row0_r
- D34 pad 1: row1_R -> row1_r
- D35 pad 1: row1_R -> row2_r
- D36 pad 1: row1_R -> row3_r
- D37 pad 1: row2_R -> row0_r
- D38 pad 1: row2_R -> row1_r
- D39 pad 1: row2_R -> row2_r
- D4 pad 1: row0 -> row3
- D40 pad 1: row2_R -> row3_r
- D41 pad 1: row2_R -> row0_r
- D42 pad 1: row2_R -> row1_r
- D43 pad 1: MISO_R -> row2_r
- D44 pad 1: MISO_R -> row3_r
- D45 pad 1: MISO_R -> row0_r
- D46 pad 1: MISO_R -> row1_r
- D47 pad 1: MISO_R -> row2_r
- D48 pad 1: MISO_R -> row3_r
- D6 pad 1: row0 -> row1
- D7 pad 1: row1 -> row2
- D8 pad 1: row1 -> row3
- D9 pad 1: row1 -> row0
- R1 pad 2: RESET -> Net-(R1-Pad2)
- R2 pad 1: GND -> GNDA
- R2 pad 2: Net-(J6-Pad4) -> Net-(R2-Pad2)
- SW1 pad 1: RESET -> col0
- SW1 pad 2: GND -> Net-(D1-A)
Routing:
- net GNDA: track 368.0 -> 94.2 mm, vias 11 -> 1
- net col0: track 0.00 -> 203.0 mm, vias 0 -> 2
- net col5_r: track 0.00 -> 197.6 mm, vias 0 -> 2
- net MISO_R: track 192.4 -> 0.00 mm, vias 5 -> 0
- net col4_r: track 0.00 -> 183.7 mm
- net row3_r: track 0.00 -> 183.4 mm
- net row3: track 0.00 -> 180.9 mm, vias 0 -> 1
- net col1: track 0.00 -> 178.4 mm
- net row2_r: track 0.00 -> 176.8 mm
- net col2: track 0.00 -> 170.4 mm, vias 0 -> 2
- net col3_r: track 0.00 -> 162.9 mm
- net +5VA: track 237.4 -> 75.0 mm, vias 7 -> 0
- net row1_r: track 0.00 -> 155.8 mm
- net row2: track 0.00 -> 149.2 mm, vias 0 -> 1
- net col3: track 0.00 -> 148.3 mm, vias 0 -> 2
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- removed copper zone on B.Cu, net GNDA
Other:
- board size 262.5 x 106.5 mm -> 294.2 x 109.7 mm
- net class Default removed
- net class Power removed
- rule pad_to_mask_clearance: 0.051 -> 0
