File: choc/yamanami_keyboard_choc.kicad_pcb (KiCad board)
At the start: 2 copper layers, 279 x 90 mm, 118 parts, among them J10 MJ-4PP-9, J5 MJ-4PP-9, U1 ProMicro, U2 ProMicro

Commit message: 途中経過の保存
Other:
- net class Default removed
- net class Power removed
